Commit message: Replace stand-in L2 mount with the CAD mast and bracket
The Unitree L2 now sits on the designed mast: a 725 mm pole flush with
the rear plate edge, with the L2 hanging inverted under a bracket tilted
20 degrees forward, so it sees the floor ahead of the robot.

- Convert the Shapr3D exports (mm, CAD assembly frame) to metres in a
  shared l2_mast frame with tools/cad_stl_to_ros.py; re-running it on a
  converted file is refused.
- unitree_l2.xacro: new l2_mast link with the pole and bracket meshes;
  l2_mount placed from the CAD face centre; args l2_mast_x/y/z/yaw and
  l2_bracket_yaw replace l2_x..l2_yaw and l2_spacer_length.
- The cable direction (toward the pole) is provisional, set only by
  l2_bracket_yaw; recorded in STANDINS.md with what to change if it
  changes. Mast mass is a stand-in.
- Add the reference photo of the mount.

Co-Authored-By: Claude Opus 5.5 <noreply@anthropic.com>

File: src/mecanum_description/urdf/sensors/unitree_l2.xacro (robot description, xacro)
@@ -1,41 +1,56 @@
 <?xml version="1.0"?>
 <!--
-  Unitree L2 4D LiDAR: mount link, lidar frame and IMU frame.
+  Unitree L2 4D LiDAR on its mast: mast link, mount link, lidar frame and IMU frame.
   Included from mecanum.urdf.xacro when use_l2 is true (the default).
-  Frames (vendor definition, unilidar_sdk2 README "Coordinate System Definition"):
-    - Lidar frame origin: centre of the L2's bottom mounting surface.
-      +X points away from the cable outlet, +Z is normal to the bottom surface, right-handed.
-    - IMU frame: axes parallel to the lidar frame, origin at
-      (-0.007698, -0.014655, 0.00667) m in the lidar frame.
-  Tree (fixed joints, published by robot_state_publisher):
-    base_link -> l2_mount -> l2_lidar   (identity: the mount frame IS the bottom mounting face)
-                 l2_mount -> l2_imu     (vendor lidar-to-IMU offset)
-  The Unitree ROS 2 driver's cloud_frame / imu_frame parameters must be set to
-  l2_lidar / l2_imu (with the prefix, if one is used) so its messages match these frames.
-  Body geometry is from the vendor datasheet: 75 x 75 x 65 mm, 230 g.
+  Mechanical design (CAD, Shapr3D; reference: refs/mecanum_ros2_lidar_placement.jpeg):
+    - A 725 mm pole (70 x 30 mm section) stands on the chassis plate, flush with its rear
+      edge, centred left-right.
+    - On top, a bracket plate tilted 20 deg overhangs forward. The L2 hangs inverted under it:
+      its bottom mounting face is against the plate, its dome points down and 20 deg forward,
+      so it sees the floor ahead of the robot.
+    Meshes: meshes/visual/725mmpole.stl (pole) and meshes/visual/lidarsetup01.stl (bracket +
+    L2 body), converted from mm to m into the l2_mast frame by tools/cad_stl_to_ros.py.
+  Frames (all fixed joints, published by robot_state_publisher):
+    base_link -> l2_mast    origin at the centre of the pole's bottom face, x along the
+                            overhang (forward), z up. Carries the pole + bracket meshes.
+    base_link -> l2_mount   centre of the L2's bottom mounting face; z into the dome
+                            (forward-down), x along the bracket away from the pole
+                            (forward-up). Pose = mast pose + CAD offset.
+    l2_mount  -> l2_lidar   vendor point-cloud frame: l2_mount rotated by l2_bracket_yaw
+                            about z (identity with the default cable direction).
+    l2_mount  -> l2_imu     vendor IMU frame: axes parallel to l2_lidar, origin at
+                            (-0.007698, -0.014655, 0.00667) m in l2_lidar.
+  Vendor frame definition (unilidar_sdk2 README): origin at the centre of the bottom mounting
+  surface, +X away from the cable outlet, +Z normal to the bottom surface into the sensor.
+  The L2 driver (mecanum_lidar) stamps its messages with l2_lidar / l2_imu.
 -->
 <robot xmlns:xacro="http://www.ros.org/wiki/xacro">
-  <!-- Mount pose of the L2 bottom mounting face relative to base_link.
-       base_link is the chassis centre at wheel-axle height (see mecanum_robot.xacro).
-       The chassis top plate is 0.040 m above base_link, so the default z puts the L2
-       upright, centred, on a 0.10 m spacer, with the cable pointing to the rear.
-       Inverted mount example: l2_roll:=3.14159 l2_z:=<height of the mounting face>. -->
-  <!-- STAND-IN: L2 mount pose (the L2 is not mounted yet), measure the centre of the L2 bottom mounting face relative to base_link once the bracket exists -->
-  <xacro:arg name="l2_x" default="0.0"/>
-  <!-- STAND-IN: L2 mount pose (the L2 is not mounted yet), measure as for l2_x -->
-  <xacro:arg name="l2_y" default="0.0"/>
-  <!-- STAND-IN: L2 mount pose (the L2 is not mounted yet), measure as for l2_x -->
-  <xacro:arg name="l2_z" default="0.14"/>
-  <!-- STAND-IN: L2 mount orientation (upright assumed), read from the bracket CAD or measure with a level -->
-  <xacro:arg name="l2_roll" default="0.0"/>
-  <!-- STAND-IN: L2 mount orientation (level assumed), read from the bracket CAD or measure with a level -->
-  <xacro:arg name="l2_pitch" default="0.0"/>
-  <!-- STAND-IN: L2 mount yaw (cable to the rear assumed), check which way the cable outlet points -->
-  <xacro:arg name="l2_yaw" default="0.0"/>
-  <!-- STAND-IN: spacer/bracket length between the mounting face and the structure it is
-       fixed to (drawn along -Z of l2_mount), measure the real bracket; 0 disables it -->
-  <xacro:arg name="l2_spacer_length" default="0.10"/>
+  <!-- Mast placement on the chassis (design values, see the header). The default puts the
+       pole's 30 mm face flush with the rear plate edge (-0.3025 + 0.015), centred, standing
+       on the plate top 0.040 m above base_link. Pole at the front instead:
+       l2_mast_x:=0.2875 l2_mast_yaw:=3.14159 -->
+  <xacro:arg name="l2_mast_x" default="-0.2875"/>
+  <xacro:arg name="l2_mast_y" default="0.0"/>
+  <xacro:arg name="l2_mast_z" default="0.040"/>
+  <xacro:arg name="l2_mast_yaw" default="0.0"/>
+  <!-- Rotation of the L2 about its own Z on the bracket. 0 = cable outlet toward the pole,
+       so vendor +X points along the overhang. PROVISIONAL design choice (subject to change):
+       if the cable direction changes, set this (pi = cable toward the overhang tip,
+       +-pi/2 = sideways) and see STANDINS.md "Provisional design choices". -->
+  <xacro:arg name="l2_bracket_yaw" default="0.0"/>
+  <!-- From the CAD (tools/cad_stl_to_ros.py, report-l2 option), in the l2_mast frame -->
+  <xacro:property name="l2_face_x" value="0.06448"/>
+  <xacro:property name="l2_face_y" value="0.0075"/>
+  <xacro:property name="l2_face_z" value="0.74229"/>
+  <xacro:property name="l2_bracket_tilt" value="${radians(20.0)}"/>
+  <!-- Pole section and height, for the mast inertia -->
+  <xacro:property name="l2_pole_x" value="0.030"/>
+  <xacro:property name="l2_pole_y" value="0.070"/>
+  <xacro:property name="l2_pole_height" value="0.725"/>
+  <!-- STAND-IN: mast mass (pole + bracket) is unknown, weigh the assembly; 0.9 kg assumes a
+       2 mm wall aluminium tube plus the bracket plate -->
+  <xacro:property name="l2_mast_mass" value="0.9"/>
   <!-- Vendor datasheet values (not stand-ins) -->
-  <xacro:property name="l2_body_radius" value="0.0375"/>
+  <xacro:property name="l2_body_size" value="0.075"/>
   <xacro:property name="l2_body_height" value="0.065"/>
   <xacro:property name="l2_mass" value="0.230"/>
@@ -44,45 +59,65 @@
   <xacro:property name="l2_imu_y" value="-0.014655"/>
   <xacro:property name="l2_imu_z" value="0.00667"/>
-  <!-- Radius of the drawn spacer; cosmetic, also used as a collision body -->
-  <xacro:property name="l2_spacer_radius" value="0.02"/>
-  <xacro:macro name="unitree_l2" params="prefix parent xyz rpy spacer_length">
-    <joint name="${prefix}l2_mount_joint" type="fixed">
+  <xacro:property name="l2_pole_mesh" value="${mesh_dir}/725mmpole.stl"/>
+  <xacro:property name="l2_bracket_mesh" value="${mesh_dir}/lidarsetup01.stl"/>
+  <xacro:macro name="unitree_l2" params="prefix parent mast_x mast_y mast_z mast_yaw bracket_yaw">
+    <!-- L2 face position in the parent frame, and the IMU offset rotated by the bracket yaw -->
+    <xacro:property name="mount_x"
+      value="${mast_x + cos(mast_yaw) * l2_face_x - sin(mast_yaw) * l2_face_y}"/>
+    <xacro:property name="mount_y"
+      value="${mast_y + sin(mast_yaw) * l2_face_x + cos(mast_yaw) * l2_face_y}"/>
+    <xacro:property name="mount_z" value="${mast_z + l2_face_z}"/>
+    <xacro:property name="imu_x"
+      value="${cos(bracket_yaw) * l2_imu_x - sin(bracket_yaw) * l2_imu_y}"/>
+    <xacro:property name="imu_y"
+      value="${sin(bracket_yaw) * l2_imu_x + cos(bracket_yaw) * l2_imu_y}"/>
+    <!-- Pole + bracket (+ the L2 body, which is part of the bracket mesh) -->
+    <joint name="${prefix}l2_mast_joint" type="fixed">
       <parent link="${prefix}${parent}"/>
-      <child link="${prefix}l2_mount"/>
-      <origin xyz="${xyz}" rpy="${rpy}"/>
+      <child link="${prefix}l2_mast"/>
+      <origin xyz="${mast_x} ${mast_y} ${mast_z}" rpy="0 0 ${mast_yaw}"/>
     </joint>
-    <!-- Sensor body. Frame origin = centre of the bottom mounting face. -->
-    <link name="${prefix}l2_mount">
+    <link name="${prefix}l2_mast">
       <visual>
-        <origin xyz="0 0 ${l2_body_height/2}" rpy="0 0 0"/>
         <geometry>
-          <cylinder radius="${l2_body_radius}" length="${l2_body_height}"/>
+          <mesh filename="${l2_pole_mesh}"/>
+        </geometry>
+        <material name="grey"/>
+      </visual>
+      <visual>
+        <geometry>
+          <mesh filename="${l2_bracket_mesh}"/>
         </geometry>
         <material name="dark_grey"/>
       </visual>
       <collision>
-        <origin xyz="0 0 ${l2_body_height/2}" rpy="0 0 0"/>
         <geometry>
-          <cylinder radius="${l2_body_radius}" length="${l2_body_height}"/>
+          <mesh filename="${l2_pole_mesh}"/>
         </geometry>
       </collision>
-      <xacro:if value="${spacer_length > 0}">
-        <visual>
-          <origin xyz="0 0 ${-spacer_length/2}" rpy="0 0 0"/>
-          <geometry>
-            <cylinder radius="${l2_spacer_radius}" length="${spacer_length}"/>
-          </geometry>
-          <material name="grey"/>
-        </visual>
-        <collision>
-          <origin xyz="0 0 ${-spacer_length/2}" rpy="0 0 0"/>
-          <geometry>
-            <cylinder radius="${l2_spacer_radius}" length="${spacer_length}"/>
-          </geometry>
-        </collision>
-      </xacro:if>
-      <xacro:cylinder_inertia mass="${l2_mass}" radius="${l2_body_radius}" length="${l2_body_height}">
+      <collision>
+        <geometry>
+          <mesh filename="${l2_bracket_mesh}"/>
+        </geometry>
+      </collision>
+      <xacro:box_inertia mass="${l2_mast_mass}" x="${l2_pole_x}" y="${l2_pole_y}"
+        z="${l2_pole_height}">
+        <origin xyz="0 0 ${l2_pole_height/2}" rpy="0 0 0"/>
+      </xacro:box_inertia>
+    </link>
+    <!-- L2 bottom mounting face: mast pose + CAD offset (rotated by the mast yaw).
+         Orientation: inverted (roll pi), then tilted 20 deg so z points forward-down.
+         URDF rpy is Rz(yaw) Ry(pitch) Rx(roll), so the mast yaw is simply the yaw term. -->
+    <joint name="${prefix}l2_mount_joint" type="fixed">
+      <parent link="${prefix}${parent}"/>
+      <child link="${prefix}l2_mount"/>
+      <origin xyz="${mount_x} ${mount_y} ${mount_z}" rpy="${pi} ${-l2_bracket_tilt} ${mast_yaw}"/>
+    </joint>
+    <!-- Sensor mass only; the body geometry is in the bracket mesh of l2_mast -->
+    <link name="${prefix}l2_mount">
+      <xacro:box_inertia mass="${l2_mass}" x="${l2_body_size}" y="${l2_body_size}"
+        z="${l2_body_height}">
         <origin xyz="0 0 ${l2_body_height/2}" rpy="0 0 0"/>
-      </xacro:cylinder_inertia>
+      </xacro:box_inertia>
     </link>
     <!-- Point cloud frame (vendor lidar frame) -->
@@ -90,18 +125,17 @@
       <parent link="${prefix}l2_mount"/>
       <child link="${prefix}l2_lidar"/>
-      <origin xyz="0 0 0" rpy="0 0 0"/>
+      <origin xyz="0 0 0" rpy="0 0 ${bracket_yaw}"/>
     </joint>
     <link name="${prefix}l2_lidar"/>
-    <!-- Built-in 6-axis IMU frame -->
+    <!-- Built-in 6-axis IMU frame: vendor offset, expressed in l2_mount -->
     <joint name="${prefix}l2_imu_joint" type="fixed">
       <parent link="${prefix}l2_mount"/>
       <child link="${prefix}l2_imu"/>
-      <origin xyz="${l2_imu_x} ${l2_imu_y} ${l2_imu_z}" rpy="0 0 0"/>
+      <origin xyz="${imu_x} ${imu_y} ${l2_imu_z}" rpy="0 0 ${bracket_yaw}"/>
     </joint>
     <link name="${prefix}l2_imu"/>
   </xacro:macro>
   <xacro:unitree_l2 prefix="$(arg prefix)" parent="base_link"
-    xyz="$(arg l2_x) $(arg l2_y) $(arg l2_z)"
-    rpy="$(arg l2_roll) $(arg l2_pitch) $(arg l2_yaw)"
-    spacer_length="$(arg l2_spacer_length)"/>
+    mast_x="$(arg l2_mast_x)" mast_y="$(arg l2_mast_y)" mast_z="$(arg l2_mast_z)"
+    mast_yaw="$(arg l2_mast_yaw)" bracket_yaw="$(arg l2_bracket_yaw)"/>
 </robot>

File: src/mecanum_simulation/urdf/mecanum_sim.urdf.xacro (robot description, xacro)
@@ -2,5 +2,5 @@
 <!--
   Simulation entry point: the unmodified robot description plus Gazebo-only additions.
-  All xacro args of mecanum_description pass through (prefix, use_l2, l2_x ... l2_spacer_length).
+  All xacro args of mecanum_description pass through (prefix, use_l2, l2_mast_x/y/z/yaw, l2_bracket_yaw).
   The sim plugins assume prefix:="" and the model name "mecanum" (see mecanum.gazebo.xacro).
 -->

Commit message: Correct the L2 mast: 810 mm pole, 30° bracket, cable at 22.9°
The committed mast model was stale. Replace it with the re-exported CAD:

- 810mmL2stand.stl (pole) and L2lidar30degree.stl (bracket + L2 block),
  converted from mm to the l2_mast frame with tools/cad_stl_to_ros.py;
  the old 725 mm / 20° meshes are removed.
- L2 face centre (0.06592, 0.0075, 0.83999) m in l2_mast, bracket tilt
  30°: l2_lidar is 0.93 m above the floor, axis 30° forward of vertical.
- l2_bracket_yaw defaults to 22.9° (0.3996804 rad): on the actual mount
  the cable exits 22.9° clockwise seen from above, toward the rear-left,
  so vendor +X points forward-right.
- README, STANDINS.md and the converter docstring updated.

Co-Authored-By: Claude Opus 5.5 <noreply@anthropic.com>

File: src/mecanum_description/urdf/sensors/unitree_l2.xacro (robot description, xacro)
@@ -4,10 +4,12 @@
   Included from mecanum.urdf.xacro when use_l2 is true (the default).
   Mechanical design (CAD, Shapr3D; reference: refs/mecanum_ros2_lidar_placement.jpeg):
-    - A 725 mm pole (70 x 30 mm section) stands on the chassis plate, flush with its rear
+    - An 810 mm pole (70 x 30 mm section) stands on the chassis plate, flush with its rear
       edge, centred left-right.
-    - On top, a bracket plate tilted 20 deg overhangs forward. The L2 hangs inverted under it:
-      its bottom mounting face is against the plate, its dome points down and 20 deg forward,
+    - On top, a bracket plate tilted 30 deg overhangs forward. The L2 hangs inverted under it:
+      its bottom mounting face is against the plate, its dome points down and 30 deg forward,
       so it sees the floor ahead of the robot.
-    Meshes: meshes/visual/725mmpole.stl (pole) and meshes/visual/lidarsetup01.stl (bracket +
+    - The L2's cable exits 22.9 deg clockwise (seen from above) from pointing straight at the
+      pole, i.e. toward the rear-left; see l2_bracket_yaw.
+    Meshes: meshes/visual/810mmL2stand.stl (pole) and meshes/visual/L2lidar30degree.stl (bracket +
     L2 body), converted from mm to m into the l2_mast frame by tools/cad_stl_to_ros.py.
   Frames (all fixed joints, published by robot_state_publisher):
@@ -18,5 +20,5 @@
                             (forward-up). Pose = mast pose + CAD offset.
     l2_mount  -> l2_lidar   vendor point-cloud frame: l2_mount rotated by l2_bracket_yaw
-                            about z (identity with the default cable direction).
+                            about z (22.9 deg on the actual mount).
     l2_mount  -> l2_imu     vendor IMU frame: axes parallel to l2_lidar, origin at
                             (-0.007698, -0.014655, 0.00667) m in l2_lidar.
@@ -34,18 +36,21 @@
   <xacro:arg name="l2_mast_z" default="0.040"/>
   <xacro:arg name="l2_mast_yaw" default="0.0"/>
-  <!-- Rotation of the L2 about its own Z on the bracket. 0 = cable outlet toward the pole,
-       so vendor +X points along the overhang. PROVISIONAL design choice (subject to change):
-       if the cable direction changes, set this (pi = cable toward the overhang tip,
-       +-pi/2 = sideways) and see STANDINS.md "Provisional design choices". -->
-  <xacro:arg name="l2_bracket_yaw" default="0.0"/>
+  <!-- Rotation (rad) of the L2 about its own Z on the bracket, from the reference orientation
+       in which the cable outlet points straight at the pole (vendor +X along the overhang).
+       The L2 hangs inverted, so its Z points down: a positive angle looks CLOCKWISE from above.
+       Actual mount: the cable exits 22.9 deg clockwise from above (toward the rear-left), so
+       vendor +X points forward-right: 0.3996804 rad = 22.9 deg. If the cable direction
+       changes, set this and see STANDINS.md "Provisional design choices"
+       (pi = cable toward the overhang tip). -->
+  <xacro:arg name="l2_bracket_yaw" default="0.3996804"/>
   <!-- From the CAD (tools/cad_stl_to_ros.py, report-l2 option), in the l2_mast frame -->
-  <xacro:property name="l2_face_x" value="0.06448"/>
+  <xacro:property name="l2_face_x" value="0.06592"/>
   <xacro:property name="l2_face_y" value="0.0075"/>
-  <xacro:property name="l2_face_z" value="0.74229"/>
-  <xacro:property name="l2_bracket_tilt" value="${radians(20.0)}"/>
+  <xacro:property name="l2_face_z" value="0.83999"/>
+  <xacro:property name="l2_bracket_tilt" value="${radians(30.0)}"/>
   <!-- Pole section and height, for the mast inertia -->
   <xacro:property name="l2_pole_x" value="0.030"/>
   <xacro:property name="l2_pole_y" value="0.070"/>
-  <xacro:property name="l2_pole_height" value="0.725"/>
+  <xacro:property name="l2_pole_height" value="0.810"/>
   <!-- STAND-IN: mast mass (pole + bracket) is unknown, weigh the assembly; 0.9 kg assumes a
        2 mm wall aluminium tube plus the bracket plate -->
@@ -59,6 +64,6 @@
   <xacro:property name="l2_imu_y" value="-0.014655"/>
   <xacro:property name="l2_imu_z" value="0.00667"/>
-  <xacro:property name="l2_pole_mesh" value="${mesh_dir}/725mmpole.stl"/>
-  <xacro:property name="l2_bracket_mesh" value="${mesh_dir}/lidarsetup01.stl"/>
+  <xacro:property name="l2_pole_mesh" value="${mesh_dir}/810mmL2stand.stl"/>
+  <xacro:property name="l2_bracket_mesh" value="${mesh_dir}/L2lidar30degree.stl"/>
   <xacro:macro name="unitree_l2" params="prefix parent mast_x mast_y mast_z mast_yaw bracket_yaw">
     <!-- L2 face position in the parent frame, and the IMU offset rotated by the bracket yaw -->
@@ -107,5 +112,5 @@
     </link>
     <!-- L2 bottom mounting face: mast pose + CAD offset (rotated by the mast yaw).
-         Orientation: inverted (roll pi), then tilted 20 deg so z points forward-down.
+         Orientation: inverted (roll pi), then tilted 30 deg so z points forward-down.
          URDF rpy is Rz(yaw) Ry(pitch) Rx(roll), so the mast yaw is simply the yaw term. -->
     <joint name="${prefix}l2_mount_joint" type="fixed">
