Commit message: Strip the current robot model for the model-v2 rewrite
The robot is getting a new model with new meshes, geometry and
additional sensors. Remove the previous model's meshes, dimensions,
masses and L2 mast so nothing silently reuses them:

- mecanum_description: delete the STL meshes and the mount photo. The
  URDF becomes a frame skeleton (names and tree kept, no meshes, poses,
  sizes or masses); unitree_l2.xacro keeps only the L2's vendor values,
  with l2_imu now under l2_lidar at the vendor offset.
- esp32_driver: remove wheel_radius/lx/ly from the YAML and the code
  defaults; the node now refuses to start until they are set.
- self_filter.yaml: remove the box (pcl_ros falls back to its +-1 m
  default until it is set again).
- test_urdf_defaults.py: skip until the new URDF exists; drop the
  code-defaults check.
- REWRITE: markers at every affected spot, a REWRITE banner on stale
  docs, and REWRITE.md listing what was removed, what to re-check and
  where the additional sensors plug in. STANDINS.md rows for removed
  values moved there.

Co-Authored-By: Claude Opus 5.5 <noreply@anthropic.com>

File: src/mecanum_description/urdf/mecanum.urdf.xacro (robot description, xacro)
@@ -10,9 +10,11 @@
   <xacro:include filename="$(find mecanum_description)/urdf/mecanum_robot.xacro"/>
   <xacro:mecanum_robot prefix="$(arg prefix)"/>
-  <!-- Unitree L2 LiDAR (mount, lidar and IMU frames). Mount pose args are declared in
-       sensors/unitree_l2.xacro. Set use_l2:=false to build the bare base. -->
+  <!-- Unitree L2 LiDAR (mount, lidar and IMU frames). Set use_l2:=false to build the bare
+       base. -->
   <xacro:arg name="use_l2" default="true"/>
   <xacro:if value="$(arg use_l2)">
     <xacro:include filename="$(find mecanum_description)/urdf/sensors/unitree_l2.xacro"/>
   </xacro:if>
+  <!-- REWRITE: include the new model's additional sensors here, one xacro per sensor in
+       urdf/sensors/ (see REWRITE.md "Where the additional sensors plug in"). -->
 </robot>

File: src/mecanum_description/urdf/mecanum_params.xacro (robot description, xacro)
@@ -1,40 +1,16 @@
 <?xml version="1.0"?>
 <!-- Physical parameters of the mecanum robot. All units SI (m, kg, rad). -->
-<!-- Dimensions match the STL meshes in meshes/visual. They combine CAD values and measured
-     approximations; the STAND-IN notes say how to measure each one (also in STANDINS.md). -->
+<!-- REWRITE: the previous model's dimensions, masses and mesh paths were removed for the new
+     model (branch feature/model-v2, see REWRITE.md). Define them here again from the new meshes
+     and geometry. Other packages consume them:
+       - wheel radius: base_joint height (base_footprint on the floor), wheel collision and
+         inertia, and wheel_radius in mecanum_base/config/esp32_driver.yaml
+       - front/rear axle x and track width: wheel joint origins, and lx (half wheelbase) and ly
+         (half track) in esp32_driver.yaml
+       - chassis extent, including every mount and sensor: the self-filter box in
+         mecanum_localization/config/self_filter.yaml and the planned Nav2 footprint
+       - masses and inertias: simulation dynamics only
+       - visual and collision mesh paths: meshes/visual and meshes/collision
+     Mark uncertain values with STAND-IN comments and list them in STANDINS.md. -->
 <robot xmlns:xacro="http://www.ros.org/wiki/xacro">
-  <!-- Chassis -->
-  <!-- STAND-IN: base plate size is approximate, measure the plate. Sets the footprint and the
-       self-filter box. -->
-  <xacro:property name="chassis_length" value="0.605"/>
-  <xacro:property name="chassis_width" value="0.394"/>
-  <xacro:property name="chassis_height" value="0.064"/>
-  <!-- STAND-IN: mass is a guess, weigh the base without wheels. Affects sim dynamics only. -->
-  <xacro:property name="chassis_mass" value="5.0"/>
-  <!-- Height of the chassis centre above base_link (wheel axle height) -->
-  <xacro:property name="chassis_z_offset" value="0.008"/>
-  <!-- Wheels -->
-  <!-- STAND-IN: effective radius under load is unknown, roll ten revolutions on the floor and
-       divide the distance by 20*pi. -->
-  <xacro:property name="wheel_radius" value="0.05"/>
-  <xacro:property name="wheel_width" value="0.08"/>
-  <!-- STAND-IN: mass is a guess, weigh one wheel with its motor mount. Sim dynamics only. -->
-  <xacro:property name="wheel_mass" value="0.3"/>
-  <!-- Wheel placement relative to base_link (chassis centre). Axles are not symmetric
-       about the chassis centre; values taken from the axle bosses on the chassis mesh. -->
-  <!-- STAND-IN: axle positions are from the mesh, measure the axle centres from the chassis
-       centre. Their difference is the wheelbase; half of it is lx in the kinematics. -->
-  <xacro:property name="front_axle_x" value="0.216"/>
-  <xacro:property name="rear_axle_x" value="-0.235"/>
-  <xacro:property name="wheelbase" value="${front_axle_x - rear_axle_x}"/>
-  <!-- track = left/right wheel centre distance -->
-  <!-- STAND-IN: track is from the mesh, measure between the wheel mid-planes. Half of it is ly
-       in the kinematics. -->
-  <xacro:property name="track_width" value="0.414"/>
-  <!-- Meshes (already in metres, origin at the link frame) -->
-  <xacro:property name="mesh_dir" value="package://mecanum_description/meshes/visual"/>
-  <xacro:property name="chassis_mesh" value="${mesh_dir}/macchumwheel_body_001_nowheel.stl"/>
-  <!-- X-configuration: diagonal wheels share the same roller handedness -->
-  <xacro:property name="wheel_mesh_left_hand" value="${mesh_dir}/macchumwheelFL.stl"/>
-  <xacro:property name="wheel_mesh_right_hand" value="${mesh_dir}/macchumwheelbase_FR.stl"/>
 </robot>

File: src/mecanum_description/urdf/mecanum_robot.xacro (robot description, xacro)
@@ -1,4 +1,8 @@
 <?xml version="1.0"?>
 <!-- Robot body: base_footprint, base_link (chassis) and the four wheels. -->
+<!-- REWRITE: frame skeleton only. The previous model's chassis mesh, collision box, inertia,
+     wheel meshes and wheel positions were removed (see REWRITE.md). The link and joint names are
+     kept because other packages use them. Rename them only together with REWRITE.md
+     "Kept, re-check after the rewrite". -->
 <robot xmlns:xacro="http://www.ros.org/wiki/xacro">
   <xacro:macro name="mecanum_robot" params="prefix">
@@ -8,35 +12,17 @@
       <parent link="${prefix}base_footprint" />
       <child link="${prefix}base_link" />
-      <origin xyz="0 0 ${wheel_radius}" rpy="0 0 0" />
+      <!-- REWRITE: origin removed. Lift base_link to the new wheel axle height (z = wheel
+           radius) so base_footprint stays on the floor. -->
     </joint>
     <!-- base_link sits at wheel axle height -->
-    <link name="${prefix}base_link">
-      <visual>
-        <origin xyz="0 0 0" rpy="0 0 0" />
-        <geometry>
-          <mesh filename="${chassis_mesh}" />
-        </geometry>
-        <material name="blue" />
-      </visual>
-      <collision>
-        <origin xyz="0 0 ${chassis_z_offset}" rpy="0 0 0" />
-        <geometry>
-          <box size="${chassis_length} ${chassis_width} ${chassis_height}" />
-        </geometry>
-      </collision>
-      <xacro:box_inertia mass="${chassis_mass}" x="${chassis_length}" y="${chassis_width}"
-        z="${chassis_height}">
-        <origin xyz="0 0 ${chassis_z_offset}" rpy="0 0 0" />
-      </xacro:box_inertia>
-    </link>
-    <!-- Wheels: left/right meshes are shared between front and rear -->
-    <xacro:mecanum_wheel prefix="${prefix}" name="front_left" parent="base_link"
-      mesh="${wheel_mesh_left_hand}" x="${front_axle_x}" y="${track_width/2}" />
-    <xacro:mecanum_wheel prefix="${prefix}" name="front_right" parent="base_link"
-      mesh="${wheel_mesh_right_hand}" x="${front_axle_x}" y="${-track_width/2}" />
-    <xacro:mecanum_wheel prefix="${prefix}" name="rear_left" parent="base_link"
-      mesh="${wheel_mesh_left_hand}" x="${rear_axle_x}" y="${track_width/2}" />
-    <xacro:mecanum_wheel prefix="${prefix}" name="rear_right" parent="base_link"
-      mesh="${wheel_mesh_right_hand}" x="${rear_axle_x}" y="${-track_width/2}" />
+    <!-- REWRITE: visual, collision and inertial removed. Add them from the new chassis meshes
+         (meshes/visual, meshes/collision), including the new geometry meshes. -->
+    <link name="${prefix}base_link" />
+    <!-- REWRITE: wheel meshes and positions removed. Pass the new wheel meshes and the wheel
+         centres (front/rear axle x, +-track/2) once mecanum_params.xacro defines them. -->
+    <xacro:mecanum_wheel prefix="${prefix}" name="front_left" parent="base_link" />
+    <xacro:mecanum_wheel prefix="${prefix}" name="front_right" parent="base_link" />
+    <xacro:mecanum_wheel prefix="${prefix}" name="rear_left" parent="base_link" />
+    <xacro:mecanum_wheel prefix="${prefix}" name="rear_right" parent="base_link" />
   </xacro:macro>
 </robot>

File: src/mecanum_description/urdf/mecanum_wheel.xacro (robot description, xacro)
@@ -1,4 +1,6 @@
 <?xml version="1.0"?>
-<!-- A single mecanum wheel: mesh visual, cylinder collision. -->
+<!-- A single mecanum wheel: link and continuous joint. -->
+<!-- REWRITE: frame skeleton only. The previous mesh visual, cylinder collision, inertia and the
+     mesh and x, y, z macro parameters were removed (see REWRITE.md). -->
 <robot xmlns:xacro="http://www.ros.org/wiki/xacro">
   <!--
@@ -6,30 +8,14 @@
     name:     wheel position, e.g. "front_left"
     parent:   link the wheel attaches to
-    mesh:     visual mesh (roller handedness)
-    x, y, z:  wheel centre relative to parent
   -->
-  <xacro:macro name="mecanum_wheel" params="prefix name parent mesh x y z:=0.0">
-    <link name="${prefix}${name}_wheel_link">
-      <visual>
-        <origin xyz="0 0 0" rpy="0 0 0"/>
-        <geometry>
-          <mesh filename="${mesh}"/>
-        </geometry>
-        <material name="dark_grey"/>
-      </visual>
-      <collision>
-        <origin xyz="0 0 0" rpy="${pi/2} 0 0"/>
-        <geometry>
-          <cylinder radius="${wheel_radius}" length="${wheel_width}"/>
-        </geometry>
-      </collision>
-      <xacro:cylinder_inertia mass="${wheel_mass}" radius="${wheel_radius}" length="${wheel_width}">
-        <origin xyz="0 0 0" rpy="${pi/2} 0 0"/>
-      </xacro:cylinder_inertia>
-    </link>
+  <xacro:macro name="mecanum_wheel" params="prefix name parent">
+    <!-- REWRITE: visual, collision and inertial from the new wheel meshes. Keep exactly one
+         unnamed collision per wheel link: the Gazebo friction block in
+         mecanum_simulation/urdf/mecanum.gazebo.xacro merges into it by name. -->
+    <link name="${prefix}${name}_wheel_link"/>
     <joint name="${prefix}${name}_wheel_joint" type="continuous">
       <parent link="${prefix}${parent}"/>
       <child link="${prefix}${name}_wheel_link"/>
-      <origin xyz="${x} ${y} ${z}" rpy="0 0 0"/>
+      <!-- REWRITE: wheel centre origin removed; set it from the new geometry -->
       <axis xyz="0 1 0"/>
     </joint>

File: src/mecanum_description/urdf/sensors/unitree_l2.xacro (robot description, xacro)
@@ -1,26 +1,18 @@
 <?xml version="1.0"?>
 <!--
-  Unitree L2 4D LiDAR on its mast: mast link, mount link, lidar frame and IMU frame.
+  Unitree L2 4D LiDAR: mount link, lidar frame and IMU frame.
   Included from mecanum.urdf.xacro when use_l2 is true (the default).
-  Mechanical design (CAD, Shapr3D; reference: refs/mecanum_ros2_lidar_placement.jpeg):
-    - An 810 mm pole (70 x 30 mm section) stands on the chassis plate, flush with its rear
-      edge, centred left-right.
-    - On top, a bracket plate tilted 30 deg overhangs forward. The L2 hangs inverted under it:
-      its bottom mounting face is against the plate, its dome points down and 30 deg forward,
-      so it sees the floor ahead of the robot.
-    - The L2's cable exits 22.9 deg clockwise (seen from above) from pointing straight at the
-      pole, i.e. toward the rear-left; see l2_bracket_yaw.
-    Meshes: meshes/visual/810mmL2stand.stl (pole) and meshes/visual/L2lidar30degree.stl (bracket +
-    L2 body), converted from mm to m into the l2_mast frame by tools/cad_stl_to_ros.py.
+  REWRITE: the previous mast was removed for the new model (see REWRITE.md): the l2_mast link
+  and joint, the pole and bracket meshes, the mast pose args (l2_mast_x/y/z/yaw), the CAD face
+  offset (l2_face_x/y/z), the 30 deg bracket tilt, the cable direction (l2_bracket_yaw) and the
+  mast mass. Only vendor facts of the L2 itself are kept below. Add the new mount's links, meshes
+  and pose when the new geometry is written.
   Frames (all fixed joints, published by robot_state_publisher):
-    base_link -> l2_mast    origin at the centre of the pole's bottom face, x along the
-                            overhang (forward), z up. Carries the pole + bracket meshes.
-    base_link -> l2_mount   centre of the L2's bottom mounting face; z into the dome
-                            (forward-down), x along the bracket away from the pole
-                            (forward-up). Pose = mast pose + CAD offset.
-    l2_mount  -> l2_lidar   vendor point-cloud frame: l2_mount rotated by l2_bracket_yaw
-                            about z (22.9 deg on the actual mount).
-    l2_mount  -> l2_imu     vendor IMU frame: axes parallel to l2_lidar, origin at
-                            (-0.007698, -0.014655, 0.00667) m in l2_lidar.
+    <parent> -> l2_mount   centre of the L2's bottom mounting face, z normal to it into the
+                           sensor (dome). REWRITE: pose on the new mount.
+    l2_mount -> l2_lidar   vendor point-cloud frame. REWRITE: rotation about z that sets the
+                           cable outlet direction on the new mount.
+    l2_lidar -> l2_imu     vendor IMU frame: axes parallel to l2_lidar, origin at
+                           (-0.007698, -0.014655, 0.00667) m in l2_lidar.
   Vendor frame definition (unilidar_sdk2 README): origin at the centre of the bottom mounting
   surface, +X away from the cable outlet, +Z normal to the bottom surface into the sensor.
@@ -28,32 +20,4 @@
 -->
 <robot xmlns:xacro="http://www.ros.org/wiki/xacro">
-  <!-- Mast placement on the chassis (design values, see the header). The default puts the
-       pole's 30 mm face flush with the rear plate edge (-0.3025 + 0.015), centred, standing
-       on the plate top 0.040 m above base_link. Pole at the front instead:
-       l2_mast_x:=0.2875 l2_mast_yaw:=3.14159 -->
-  <xacro:arg name="l2_mast_x" default="-0.2875"/>
-  <xacro:arg name="l2_mast_y" default="0.0"/>
-  <xacro:arg name="l2_mast_z" default="0.040"/>
-  <xacro:arg name="l2_mast_yaw" default="0.0"/>
-  <!-- Rotation (rad) of the L2 about its own Z on the bracket, from the reference orientation
-       in which the cable outlet points straight at the pole (vendor +X along the overhang).
-       The L2 hangs inverted, so its Z points down: a positive angle looks CLOCKWISE from above.
-       Actual mount: the cable exits 22.9 deg clockwise from above (toward the rear-left), so
-       vendor +X points forward-right: 0.3996804 rad = 22.9 deg. If the cable direction
-       changes, set this and see STANDINS.md "Provisional design choices"
-       (pi = cable toward the overhang tip). -->
-  <xacro:arg name="l2_bracket_yaw" default="0.3996804"/>
-  <!-- From the CAD (tools/cad_stl_to_ros.py, report-l2 option), in the l2_mast frame -->
-  <xacro:property name="l2_face_x" value="0.06592"/>
-  <xacro:property name="l2_face_y" value="0.0075"/>
-  <xacro:property name="l2_face_z" value="0.83999"/>
-  <xacro:property name="l2_bracket_tilt" value="${radians(30.0)}"/>
-  <!-- Pole section and height, for the mast inertia -->
-  <xacro:property name="l2_pole_x" value="0.030"/>
-  <xacro:property name="l2_pole_y" value="0.070"/>
-  <xacro:property name="l2_pole_height" value="0.810"/>
-  <!-- STAND-IN: mast mass (pole + bracket) is unknown, weigh the assembly; 0.9 kg assumes a
-       2 mm wall aluminium tube plus the bracket plate -->
-  <xacro:property name="l2_mast_mass" value="0.9"/>
   <!-- Vendor datasheet values (not stand-ins) -->
   <xacro:property name="l2_body_size" value="0.075"/>
@@ -64,60 +28,13 @@
   <xacro:property name="l2_imu_y" value="-0.014655"/>
   <xacro:property name="l2_imu_z" value="0.00667"/>
-  <xacro:property name="l2_pole_mesh" value="${mesh_dir}/810mmL2stand.stl"/>
-  <xacro:property name="l2_bracket_mesh" value="${mesh_dir}/L2lidar30degree.stl"/>
-  <xacro:macro name="unitree_l2" params="prefix parent mast_x mast_y mast_z mast_yaw bracket_yaw">
-    <!-- L2 face position in the parent frame, and the IMU offset rotated by the bracket yaw -->
-    <xacro:property name="mount_x"
-      value="${mast_x + cos(mast_yaw) * l2_face_x - sin(mast_yaw) * l2_face_y}"/>
-    <xacro:property name="mount_y"
-      value="${mast_y + sin(mast_yaw) * l2_face_x + cos(mast_yaw) * l2_face_y}"/>
-    <xacro:property name="mount_z" value="${mast_z + l2_face_z}"/>
-    <xacro:property name="imu_x"
-      value="${cos(bracket_yaw) * l2_imu_x - sin(bracket_yaw) * l2_imu_y}"/>
-    <xacro:property name="imu_y"
-      value="${sin(bracket_yaw) * l2_imu_x + cos(bracket_yaw) * l2_imu_y}"/>
-    <!-- Pole + bracket (+ the L2 body, which is part of the bracket mesh) -->
-    <joint name="${prefix}l2_mast_joint" type="fixed">
-      <parent link="${prefix}${parent}"/>
-      <child link="${prefix}l2_mast"/>
-      <origin xyz="${mast_x} ${mast_y} ${mast_z}" rpy="0 0 ${mast_yaw}"/>
-    </joint>
-    <link name="${prefix}l2_mast">
-      <visual>
-        <geometry>
-          <mesh filename="${l2_pole_mesh}"/>
-        </geometry>
-        <material name="grey"/>
-      </visual>
-      <visual>
-        <geometry>
-          <mesh filename="${l2_bracket_mesh}"/>
-        </geometry>
-        <material name="dark_grey"/>
-      </visual>
-      <collision>
-        <geometry>
-          <mesh filename="${l2_pole_mesh}"/>
-        </geometry>
-      </collision>
-      <collision>
-        <geometry>
-          <mesh filename="${l2_bracket_mesh}"/>
-        </geometry>
-      </collision>
-      <xacro:box_inertia mass="${l2_mast_mass}" x="${l2_pole_x}" y="${l2_pole_y}"
-        z="${l2_pole_height}">
-        <origin xyz="0 0 ${l2_pole_height/2}" rpy="0 0 0"/>
-      </xacro:box_inertia>
-    </link>
-    <!-- L2 bottom mounting face: mast pose + CAD offset (rotated by the mast yaw).
-         Orientation: inverted (roll pi), then tilted 30 deg so z points forward-down.
-         URDF rpy is Rz(yaw) Ry(pitch) Rx(roll), so the mast yaw is simply the yaw term. -->
+  <xacro:macro name="unitree_l2" params="prefix parent">
     <joint name="${prefix}l2_mount_joint" type="fixed">
       <parent link="${prefix}${parent}"/>
       <child link="${prefix}l2_mount"/>
-      <origin xyz="${mount_x} ${mount_y} ${mount_z}" rpy="${pi} ${-l2_bracket_tilt} ${mast_yaw}"/>
+      <!-- REWRITE: origin removed. Set the L2's bottom mounting face pose on the new mount
+           (position, tilt, z into the dome). -->
     </joint>
-    <!-- Sensor mass only; the body geometry is in the bracket mesh of l2_mast -->
+    <!-- Sensor mass only. REWRITE: add the L2 body visual/collision, unless the new mount's
+         meshes already contain it. -->
     <link name="${prefix}l2_mount">
       <xacro:box_inertia mass="${l2_mass}" x="${l2_body_size}" y="${l2_body_size}"
@@ -130,17 +47,17 @@
       <parent link="${prefix}l2_mount"/>
       <child link="${prefix}l2_lidar"/>
-      <origin xyz="0 0 0" rpy="0 0 ${bracket_yaw}"/>
+      <!-- REWRITE: rotation removed. Rotate about z so vendor +X points away from the cable
+           outlet as mounted on the new robot. -->
     </joint>
     <link name="${prefix}l2_lidar"/>
-    <!-- Built-in 6-axis IMU frame: vendor offset, expressed in l2_mount -->
+    <!-- Built-in 6-axis IMU frame: vendor offset in the lidar frame -->
     <joint name="${prefix}l2_imu_joint" type="fixed">
-      <parent link="${prefix}l2_mount"/>
+      <parent link="${prefix}l2_lidar"/>
       <child link="${prefix}l2_imu"/>
-      <origin xyz="${imu_x} ${imu_y} ${l2_imu_z}" rpy="0 0 ${bracket_yaw}"/>
+      <origin xyz="${l2_imu_x} ${l2_imu_y} ${l2_imu_z}" rpy="0 0 0"/>
     </joint>
     <link name="${prefix}l2_imu"/>
   </xacro:macro>
-  <xacro:unitree_l2 prefix="$(arg prefix)" parent="base_link"
-    mast_x="$(arg l2_mast_x)" mast_y="$(arg l2_mast_y)" mast_z="$(arg l2_mast_z)"
-    mast_yaw="$(arg l2_mast_yaw)" bracket_yaw="$(arg l2_bracket_yaw)"/>
+  <!-- REWRITE: parent is base_link until the new mount's links exist -->
+  <xacro:unitree_l2 prefix="$(arg prefix)" parent="base_link"/>
 </robot>

File: src/mecanum_simulation/urdf/mecanum.gazebo.xacro (robot description, xacro)
@@ -11,4 +11,7 @@
      X-roller layout: front_left and rear_right rollers along (1, -1); front_right and
      rear_left along (1, 1).
+     REWRITE: the fdir values below assume the previous wheels' roller handedness. Check them
+     against the new wheel meshes. The new wheel links need exactly one unnamed collision each,
+     or this friction block no longer merges and the wheels lose their mecanum behaviour.
   2. One JointController (velocity mode) per wheel. Its gz topic is the default
      /model/mecanum/joint/<joint>/cmd_vel (gz.msgs.Double, rad/s), bridged from
@@ -60,4 +63,6 @@
        elevation 0..90 deg in standard mode (factory default, work-mode bit 0 = 0) or
        -6..90 deg in wide mode (bit 0 = 1). -->
+  <!-- The sensor model below is the L2's own and carries over to the new model; its pose
+       follows l2_lidar / l2_imu from the URDF. -->
   <xacro:arg name="sim_l2_wide_fov" default="false"/>
   <xacro:if value="$(arg use_l2)">
@@ -137,4 +142,6 @@
   </gazebo>
   </xacro:if>
+  <!-- REWRITE: add Gazebo sensors for the new model's additional sensors here, on their URDF
+       frames, and bridge them in config/gz_bridge.yaml (see REWRITE.md). -->
   <gazebo>
     <plugin filename="gz-sim-odometry-publisher-system"

File: src/mecanum_simulation/urdf/mecanum_sim.urdf.xacro (robot description, xacro)
@@ -2,5 +2,5 @@
 <!--
   Simulation entry point: the unmodified robot description plus Gazebo-only additions.
-  All xacro args of mecanum_description pass through (prefix, use_l2, l2_mast_x/y/z/yaw, l2_bracket_yaw).
+  All xacro args of mecanum_description pass through (prefix, use_l2).
   The sim plugins assume prefix:="" and the model name "mecanum" (see mecanum.gazebo.xacro).
 -->
