Commit message: Add model v2 description and the sim-only plan (phase 0)
Rebuild the robot model from the reference URDF and redo the plan
around the new sensors and the wheel encoders:

- mecanum_description: model v2 from refs/washroom_robot.urdf
  (chassis_link with 18 boxes, 0.1025 m wheels, masses and inertia),
  the upright L2 on its 30 mm standoff, and one xacro per new sensor
  (D435i, RPLIDAR C1, ultrasonics, cliff ToF, bumpers) behind use_*
  args. test_reference_urdf.py checks every frame against the
  reference; the RViz configs list the new links.
- Restore the values removed in the strip: driver geometry
  (wheel_radius 0.1025, lx 0.2360, ly 0.2150), the self-filter box,
  and test_urdf_defaults. Resolve every REWRITE marker and delete
  REWRITE.md; new stand-ins go to STANDINS.md.
- Sim: the L2 defaults to wide mode; the restroom world is open on
  top in the GUI with translucent outer walls (sensors unaffected).
- tools: l2_mount_check fits the ceiling for the upright mount;
  cad_stl_to_ros drops the old mast report.
- docs: plan.md rewritten as a sim-only build, phases 0-8 (ros2_control,
  sensor suite, EKF, safety, slam_toolbox on the C1, Nav2, docking);
  hardware docs, encoder guide and READMEs updated for the new model;
  decision 0001 marked superseded. Add the sensor/BOM PDF and the
  CAD-vs-URDF image.
- Stop tracking __pycache__ files.

Co-Authored-By: Claude Opus 5.5 <noreply@anthropic.com>

File: src/mecanum_description/urdf/materials.xacro (robot description, xacro)
@@ -1,15 +1,38 @@
 <?xml version="1.0"?>
+<!-- RViz colours. The sensor colours match the callouts in
+     docs/Washroom_Robot_Prototype_Sensors_and_BOM.pdf. -->
 <robot xmlns:xacro="http://www.ros.org/wiki/xacro">
-  <material name="grey">
-    <color rgba="0.5 0.5 0.5 1.0"/>
+  <material name="cad_grey">
+    <color rgba="0.352 0.352 0.371 1"/>
   </material>
-  <material name="dark_grey">
-    <color rgba="0.2 0.2 0.2 1.0"/>
+  <material name="tyre_black">
+    <color rgba="0.1 0.1 0.1 1"/>
   </material>
-  <material name="blue">
-    <color rgba="0.1 0.3 0.8 1.0"/>
+  <material name="hub_grey">
+    <color rgba="0.55 0.55 0.58 1"/>
   </material>
-  <material name="orange">
-    <color rgba="1.0 0.5 0.0 1.0"/>
+  <material name="marker_white">
+    <color rgba="0.92 0.92 0.92 1"/>
+  </material>
+  <material name="l2_purple">
+    <color rgba="0.48 0.45 0.85 1"/>
+  </material>
+  <material name="mount_white">
+    <color rgba="0.85 0.85 0.85 1"/>
+  </material>
+  <material name="d435i_green">
+    <color rgba="0.12 0.62 0.47 1"/>
+  </material>
+  <material name="lidar_orange">
+    <color rgba="0.85 0.37 0.19 1"/>
+  </material>
+  <material name="ultrasonic_ochre">
+    <color rgba="0.72 0.46 0.1 1"/>
+  </material>
+  <material name="tof_blue">
+    <color rgba="0.23 0.53 0.84 1"/>
+  </material>
+  <material name="bumper_red">
+    <color rgba="0.88 0.28 0.28 1"/>
   </material>
 </robot>

File: src/mecanum_description/urdf/mecanum.urdf.xacro (robot description, xacro)
@@ -1,4 +1,4 @@
 <?xml version="1.0"?>
-<!-- Main entry point for the mecanum robot description. -->
+<!-- Main entry point for the mecanum robot description (the washroom robot prototype). -->
 <robot name="mecanum" xmlns:xacro="http://www.ros.org/wiki/xacro">
   <!-- Optional prefix for all links/joints (e.g. "robot1_") -->
@@ -10,11 +10,36 @@
   <xacro:include filename="$(find mecanum_description)/urdf/mecanum_robot.xacro"/>
   <xacro:mecanum_robot prefix="$(arg prefix)"/>
-  <!-- Unitree L2 LiDAR (mount, lidar and IMU frames). Set use_l2:=false to build the bare
-       base. -->
+  <!-- Sensors, one xacro each in urdf/sensors/. Set use_<sensor>:=false to leave one out. -->
+  <!-- Unitree L2 LiDAR (mount, lidar and IMU frames) -->
   <xacro:arg name="use_l2" default="true"/>
   <xacro:if value="$(arg use_l2)">
     <xacro:include filename="$(find mecanum_description)/urdf/sensors/unitree_l2.xacro"/>
   </xacro:if>
-  <!-- REWRITE: include the new model's additional sensors here, one xacro per sensor in
-       urdf/sensors/ (see REWRITE.md "Where the additional sensors plug in"). -->
+  <!-- RealSense D435i depth camera (body and optical frames) -->
+  <xacro:arg name="use_d435i" default="true"/>
+  <xacro:if value="$(arg use_d435i)">
+    <xacro:include filename="$(find mecanum_description)/urdf/sensors/realsense_d435i.xacro"/>
+  </xacro:if>
+  <!-- RPLIDAR C1 2D lidar (scan frame) -->
+  <xacro:arg name="use_lidar_2d" default="true"/>
+  <xacro:if value="$(arg use_lidar_2d)">
+    <xacro:include filename="$(find mecanum_description)/urdf/sensors/lidar_2d.xacro"/>
+  </xacro:if>
+  <!-- Four ultrasonic rangers (beam frames) -->
+  <xacro:arg name="use_ultrasonics" default="true"/>
+  <xacro:if value="$(arg use_ultrasonics)">
+    <xacro:include filename="$(find mecanum_description)/urdf/sensors/ultrasonics.xacro"/>
+  </xacro:if>
+  <!-- Four downward cliff ToF sensors (beam frames) -->
+  <xacro:arg name="use_cliff_tof" default="true"/>
+  <xacro:if value="$(arg use_cliff_tof)">
+    <xacro:include filename="$(find mecanum_description)/urdf/sensors/cliff_tof.xacro"/>
+  </xacro:if>
+  <!-- Front and rear bumper planks -->
+  <xacro:arg name="use_bumpers" default="true"/>
+  <xacro:if value="$(arg use_bumpers)">
+    <xacro:include filename="$(find mecanum_description)/urdf/sensors/bumpers.xacro"/>
+  </xacro:if>
+  <!-- Not modelled: the E-stop (rear face of the tall box), the arm (not in the CAD yet) and
+       the internal electronics. -->
 </robot>

File: src/mecanum_description/urdf/mecanum_params.xacro (robot description, xacro)
@@ -1,16 +1,49 @@
 <?xml version="1.0"?>
-<!-- Physical parameters of the mecanum robot. All units SI (m, kg, rad). -->
-<!-- REWRITE: the previous model's dimensions, masses and mesh paths were removed for the new
-     model (branch feature/model-v2, see REWRITE.md). Define them here again from the new meshes
-     and geometry. Other packages consume them:
-       - wheel radius: base_joint height (base_footprint on the floor), wheel collision and
-         inertia, and wheel_radius in mecanum_base/config/esp32_driver.yaml
-       - front/rear axle x and track width: wheel joint origins, and lx (half wheelbase) and ly
-         (half track) in esp32_driver.yaml
-       - chassis extent, including every mount and sensor: the self-filter box in
-         mecanum_localization/config/self_filter.yaml and the planned Nav2 footprint
-       - masses and inertias: simulation dynamics only
-       - visual and collision mesh paths: meshes/visual and meshes/collision
-     Mark uncertain values with STAND-IN comments and list them in STANDINS.md. -->
+<!-- Physical parameters of the robot. All units SI (m, kg, rad).
+     Source: the reference URDF refs/washroom_robot.urdf, generated from the STEP model
+     (wholerobotstepfile001.step, units mm, converted to metres there) and the sensor placement
+     PDF docs/Washroom_Robot_Prototype_Sensors_and_BOM.pdf. Where the two disagree the reference
+     URDF wins; its header lists each difference. test/test_reference_urdf.py checks that the
+     frames built from these values match the reference.
+     Frames: base_footprint on the floor below the wheel-rectangle centre; base_link directly
+     above it at wheel-axle height. Every pose below is relative to base_link.
+     Other packages consume these values:
+       - wheel_radius, front/rear_axle_x, wheel_y: wheel_radius, lx and ly in
+         mecanum_base/config/esp32_driver.yaml (checked by test_urdf_defaults.py)
+       - the body extent (including every sensor): the self-filter box in
+         mecanum_localization/config/self_filter.yaml and the Nav2 footprint
+       - masses and inertias: simulation dynamics only -->
 <robot xmlns:xacro="http://www.ros.org/wiki/xacro">
+  <!-- ===== Wheels (STEP bodies 'Folder 28*') ===== -->
+  <!-- STAND-IN: unloaded CAD radius; measure the loaded radius on the robot -->
+  <xacro:property name="wheel_radius" value="0.1025"/>
+  <xacro:property name="wheel_width" value="0.085"/>
+  <xacro:property name="wheel_hub_radius" value="0.05"/>
+  <!-- STAND-IN: no masses were supplied; 1.5 kg assumed per wheel (the drive motors are
+       counted in chassis_mass). Weigh one wheel with its hub. -->
+  <xacro:property name="wheel_mass" value="1.5"/>
+  <!-- Inertia of the STEP wheel solid scaled to wheel_mass (about the wheel centre) -->
+  <xacro:property name="wheel_ixx" value="0.00582886"/>
+  <xacro:property name="wheel_iyy" value="0.0100038"/>
+  <!-- Wheel centre of mass offset along the axle, toward the robot centreline -->
+  <xacro:property name="wheel_com_y" value="0.0003"/>
+  <!-- Wheel centres. lx = (front_axle_x - rear_axle_x) / 2 = 0.2360, ly = wheel_y = 0.2150.
+       The STEP puts the left wheels at y +0.2148 and the right ones at -0.2152 (0.2 mm off
+       centre); they are made symmetric here, as the kinematics assume. -->
+  <xacro:property name="front_axle_x" value="0.2363"/>
+  <xacro:property name="rear_axle_x" value="-0.2357"/>
+  <xacro:property name="wheel_y" value="0.2150"/>
+  <!-- ===== Body (STEP body 'Cover', rebuilt from boxes in mecanum_robot.xacro) ===== -->
+  <!-- Envelope relative to base_link: x -0.391..0.399, y -0.255..0.255,
+       z -0.0037..0.6344 (0.099..0.737 m above the floor). -->
+  <!-- STAND-IN: no masses were supplied. 25 kg = frame, panels, battery, drive motors,
+       electronics and sensors (except the L2's vendor mass), spread evenly over the envelope.
+       The real centre of mass is probably lower (battery, motors). Weigh the robot. -->
+  <xacro:property name="chassis_mass" value="25.0"/>
+  <xacro:property name="chassis_com_x" value="-0.065"/>
+  <xacro:property name="chassis_com_z" value="0.2426"/>
+  <xacro:property name="chassis_ixx" value="1.25341"/>
+  <xacro:property name="chassis_iyy" value="1.83996"/>
+  <xacro:property name="chassis_izz" value="1.69493"/>
+  <xacro:property name="chassis_ixz" value="0.331293"/>
 </robot>

File: src/mecanum_description/urdf/mecanum_robot.xacro (robot description, xacro)
@@ -1,28 +1,86 @@
 <?xml version="1.0"?>
-<!-- Robot body: base_footprint, base_link (chassis) and the four wheels. -->
-<!-- REWRITE: frame skeleton only. The previous model's chassis mesh, collision box, inertia,
-     wheel meshes and wheel positions were removed (see REWRITE.md). The link and joint names are
-     kept because other packages use them. Rename them only together with REWRITE.md
-     "Kept, re-check after the rewrite". -->
+<!-- Robot body: base_footprint, base_link, chassis_link and the four wheels. -->
+<!-- The link and joint names are used by other packages (mecanum_base WHEEL_NAMES, the Gazebo
+     friction and bridge topics, the LIO, self-filter and scan configs, the RViz files). Rename
+     them only everywhere at once. -->
 <robot xmlns:xacro="http://www.ros.org/wiki/xacro">
+  <!-- One box of the body envelope, used for both visual and collision -->
+  <xacro:macro name="chassis_box" params="xyz rpy:='0 0 0' size">
+    <visual>
+      <origin xyz="${xyz}" rpy="${rpy}"/>
+      <geometry>
+        <box size="${size}"/>
+      </geometry>
+      <material name="cad_grey"/>
+    </visual>
+    <collision>
+      <origin xyz="${xyz}" rpy="${rpy}"/>
+      <geometry>
+        <box size="${size}"/>
+      </geometry>
+    </collision>
+  </xacro:macro>
   <xacro:macro name="mecanum_robot" params="prefix">
-    <!-- Ground-projected robot frame (REP-105) -->
+    <!-- Ground-projected robot frame (REP-105), below the wheel-rectangle centre -->
     <link name="${prefix}base_footprint" />
     <joint name="${prefix}base_joint" type="fixed">
       <parent link="${prefix}base_footprint" />
       <child link="${prefix}base_link" />
-      <!-- REWRITE: origin removed. Lift base_link to the new wheel axle height (z = wheel
-           radius) so base_footprint stays on the floor. -->
+      <origin xyz="0 0 ${wheel_radius}" rpy="0 0 0" />
     </joint>
-    <!-- base_link sits at wheel axle height -->
-    <!-- REWRITE: visual, collision and inertial removed. Add them from the new chassis meshes
-         (meshes/visual, meshes/collision), including the new geometry meshes. -->
+    <!-- base_link sits at wheel axle height. Frame only: the body mass is in chassis_link, so
+         robot_state_publisher does not warn about an inertial root (Gazebo lumps the fixed
+         joint). -->
     <link name="${prefix}base_link" />
-    <!-- REWRITE: wheel meshes and positions removed. Pass the new wheel meshes and the wheel
-         centres (front/rear axle x, +-track/2) once mecanum_params.xacro defines them. -->
-    <xacro:mecanum_wheel prefix="${prefix}" name="front_left" parent="base_link" />
-    <xacro:mecanum_wheel prefix="${prefix}" name="front_right" parent="base_link" />
-    <xacro:mecanum_wheel prefix="${prefix}" name="rear_left" parent="base_link" />
-    <xacro:mecanum_wheel prefix="${prefix}" name="rear_right" parent="base_link" />
+    <!-- Outer envelope of the STEP body 'Cover', rebuilt from its planar faces as 18 boxes.
+         The rotated ones follow the 60 deg front slope and the 20 deg rear-notch floor and its
+         pad. The underside slab is split to leave an open pocket under each cliff sensor, as
+         the STEP body is open underneath. The wheel-hub profile and the bumper edge fillets
+         are simplified. -->
+    <link name="${prefix}chassis_link">
+      <inertial>
+        <origin xyz="${chassis_com_x} 0 ${chassis_com_z}" rpy="0 0 0"/>
+        <mass value="${chassis_mass}"/>
+        <inertia ixx="${chassis_ixx}" ixy="0" ixz="${chassis_ixz}" iyy="${chassis_iyy}"
+                 iyz="0" izz="${chassis_izz}"/>
+      </inertial>
+      <!-- Underside slab, 9 parts around the four cliff-sensor pockets -->
+      <xacro:chassis_box xyz="-0.3805 0 0.0224" size="0.021 0.51 0.0521"/>
+      <xacro:chassis_box xyz="-0.3535 -0.2449 0.0224" size="0.033 0.0202 0.0521"/>
+      <xacro:chassis_box xyz="-0.3535 0 0.0224" size="0.033 0.3616 0.0521"/>
+      <xacro:chassis_box xyz="-0.3535 0.2449 0.0224" size="0.033 0.0202 0.0521"/>
+      <xacro:chassis_box xyz="0 0 0.0224" size="0.674 0.51 0.0521"/>
+      <xacro:chassis_box xyz="0.3535 -0.2449 0.0224" size="0.033 0.0202 0.0521"/>
+      <xacro:chassis_box xyz="0.3535 0 0.0224" size="0.033 0.3616 0.0521"/>
+      <xacro:chassis_box xyz="0.3535 0.2449 0.0224" size="0.033 0.0202 0.0521"/>
+      <xacro:chassis_box xyz="0.3845 0 0.0224" size="0.029 0.51 0.0521"/>
+      <!-- Lower body (envelope of the open-bottom shell) -->
+      <xacro:chassis_box xyz="0.004 0 0.1446" size="0.79 0.51 0.1923"/>
+      <!-- Raised deck (the arm will stand here) -->
+      <xacro:chassis_box xyz="-0.0755 0 0.2831" size="0.6309 0.51 0.0846"/>
+      <!-- 60 deg slope from the deck down to the front step -->
+      <xacro:chassis_box xyz="0.2438 0 0.2713" rpy="0 -0.523598775 0" size="0.0473 0.51 0.0977"/>
+      <!-- Tall box: front part and the two rear ears around the rear notch -->
+      <xacro:chassis_box xyz="-0.1255 0 0.4799" size="0.167 0.51 0.309"/>
+      <xacro:chassis_box xyz="-0.3 0.1975 0.4799" size="0.182 0.115 0.309"/>
+      <xacro:chassis_box xyz="-0.3 -0.1975 0.4799" size="0.182 0.115 0.309"/>
+      <!-- Rear notch: below its floor, the 20 deg floor, and the 2 mm raised pad on it -->
+      <xacro:chassis_box xyz="-0.3 0 0.4016" size="0.182 0.28 0.1523"/>
+      <xacro:chassis_box xyz="-0.2885 0 0.4792" rpy="0 -0.349044398 0" size="0.1937 0.28 0.0672"/>
+      <xacro:chassis_box xyz="-0.2902 0 0.5149" rpy="0 -0.34906585 0" size="0.125 0.223 0.003"/>
+    </link>
+    <joint name="${prefix}chassis_joint" type="fixed">
+      <parent link="${prefix}base_link" />
+      <child link="${prefix}chassis_link" />
+      <origin xyz="0 0 0" rpy="0 0 0" />
+    </joint>
+    <xacro:mecanum_wheel prefix="${prefix}" name="front_left" parent="base_link"
+      x="${front_axle_x}" y="${wheel_y}" side="1" />
+    <xacro:mecanum_wheel prefix="${prefix}" name="front_right" parent="base_link"
+      x="${front_axle_x}" y="${-wheel_y}" side="-1" />
+    <xacro:mecanum_wheel prefix="${prefix}" name="rear_left" parent="base_link"
+      x="${rear_axle_x}" y="${wheel_y}" side="1" />
+    <xacro:mecanum_wheel prefix="${prefix}" name="rear_right" parent="base_link"
+      x="${rear_axle_x}" y="${-wheel_y}" side="-1" />
   </xacro:macro>
 </robot>

File: src/mecanum_description/urdf/mecanum_wheel.xacro (robot description, xacro)
@@ -1,6 +1,4 @@
 <?xml version="1.0"?>
 <!-- A single mecanum wheel: link and continuous joint. -->
-<!-- REWRITE: frame skeleton only. The previous mesh visual, cylinder collision, inertia and the
-     mesh and x, y, z macro parameters were removed (see REWRITE.md). -->
 <robot xmlns:xacro="http://www.ros.org/wiki/xacro">
   <!--
@@ -8,14 +6,56 @@
     name:     wheel position, e.g. "front_left"
     parent:   link the wheel attaches to
+    x, y:     wheel centre (tread mid-plane on the axle) in the parent frame
+    side:     1 for a left wheel, -1 for a right wheel
+    The joint axis is +y for all four wheels, so a positive joint velocity rolls the robot
+    forward on every wheel. The rollers are not modelled (the CAD has none): the roller
+    handedness (X layout) lives in mecanum_base/kinematics.py and the sim friction directions.
   -->
-  <xacro:macro name="mecanum_wheel" params="prefix name parent">
-    <!-- REWRITE: visual, collision and inertial from the new wheel meshes. Keep exactly one
-         unnamed collision per wheel link: the Gazebo friction block in
-         mecanum_simulation/urdf/mecanum.gazebo.xacro merges into it by name. -->
-    <link name="${prefix}${name}_wheel_link"/>
+  <xacro:macro name="mecanum_wheel" params="prefix name parent x y side">
+    <link name="${prefix}${name}_wheel_link">
+      <inertial>
+        <origin xyz="0 ${-side * wheel_com_y} 0" rpy="0 0 0"/>
+        <mass value="${wheel_mass}"/>
+        <inertia ixx="${wheel_ixx}" ixy="0" ixz="0" iyy="${wheel_iyy}" iyz="0"
+                 izz="${wheel_ixx}"/>
+      </inertial>
+      <!-- Tyre -->
+      <visual>
+        <origin xyz="0 0 0" rpy="${pi/2} 0 0"/>
+        <geometry>
+          <cylinder radius="${wheel_radius}" length="${wheel_width}"/>
+        </geometry>
+        <material name="tyre_black"/>
+      </visual>
+      <!-- Hub -->
+      <visual>
+        <origin xyz="0 0 0" rpy="${pi/2} 0 0"/>
+        <geometry>
+          <cylinder radius="${wheel_hub_radius}" length="${wheel_width + 0.002}"/>
+        </geometry>
+        <material name="hub_grey"/>
+      </visual>
+      <!-- White bar across the wheel face: shows the wheel turning in RViz -->
+      <visual>
+        <origin xyz="0 0 0" rpy="0 0 0"/>
+        <geometry>
+          <box size="0.014 ${wheel_width + 0.003} ${0.85 * 2 * wheel_radius}"/>
+        </geometry>
+        <material name="marker_white"/>
+      </visual>
+      <!-- Exactly one unnamed collision: the Gazebo friction block in
+           mecanum_simulation/urdf/mecanum.gazebo.xacro merges into it by name
+           (<link>_collision), and test_urdf_defaults.py reads its radius. -->
+      <collision>
+        <origin xyz="0 0 0" rpy="${pi/2} 0 0"/>
+        <geometry>
+          <cylinder radius="${wheel_radius}" length="${wheel_width}"/>
+        </geometry>
+      </collision>
+    </link>
     <joint name="${prefix}${name}_wheel_joint" type="continuous">
       <parent link="${prefix}${parent}"/>
       <child link="${prefix}${name}_wheel_link"/>
-      <!-- REWRITE: wheel centre origin removed; set it from the new geometry -->
+      <origin xyz="${x} ${y} 0" rpy="0 0 0"/>
       <axis xyz="0 1 0"/>
     </joint>
