Commit message: Add model v2 description and the sim-only plan (phase 0)
Rebuild the robot model from the reference URDF and redo the plan
around the new sensors and the wheel encoders:

- mecanum_description: model v2 from refs/washroom_robot.urdf
  (chassis_link with 18 boxes, 0.1025 m wheels, masses and inertia),
  the upright L2 on its 30 mm standoff, and one xacro per new sensor
  (D435i, RPLIDAR C1, ultrasonics, cliff ToF, bumpers) behind use_*
  args. test_reference_urdf.py checks every frame against the
  reference; the RViz configs list the new links.
- Restore the values removed in the strip: driver geometry
  (wheel_radius 0.1025, lx 0.2360, ly 0.2150), the self-filter box,
  and test_urdf_defaults. Resolve every REWRITE marker and delete
  REWRITE.md; new stand-ins go to STANDINS.md.
- Sim: the L2 defaults to wide mode; the restroom world is open on
  top in the GUI with translucent outer walls (sensors unaffected).
- tools: l2_mount_check fits the ceiling for the upright mount;
  cad_stl_to_ros drops the old mast report.
- docs: plan.md rewritten as a sim-only build, phases 0-8 (ros2_control,
  sensor suite, EKF, safety, slam_toolbox on the C1, Nav2, docking);
  hardware docs, encoder guide and READMEs updated for the new model;
  decision 0001 marked superseded. Add the sensor/BOM PDF and the
  CAD-vs-URDF image.
- Stop tracking __pycache__ files.

Co-Authored-By: Claude Opus 5.5 <noreply@anthropic.com>

File: src/mecanum_description/urdf/sensors/unitree_l2.xacro (robot description, xacro)
@@ -3,14 +3,17 @@
   Unitree L2 4D LiDAR: mount link, lidar frame and IMU frame.
   Included from mecanum.urdf.xacro when use_l2 is true (the default).
-  REWRITE: the previous mast was removed for the new model (see REWRITE.md): the l2_mast link
-  and joint, the pole and bracket meshes, the mast pose args (l2_mast_x/y/z/yaw), the CAD face
-  offset (l2_face_x/y/z), the 30 deg bracket tilt, the cable direction (l2_bracket_yaw) and the
-  mast mass. Only vendor facts of the L2 itself are kept below. Add the new mount's links, meshes
-  and pose when the new geometry is written.
+  Mount: upright on a 30 mm standoff on the top of the tall box, behind the robot centre
+  (PDF schedule: "box top on 30 mm standoff, upright, negative-angle mode"). The STEP model has
+  the L2 sunk 40 mm into the box top, which contradicts the PDF; the PDF mounting is used. The
+  standoff is drawn with the L2's footprint; its real shape is unknown.
+  Field of view: the hemisphere on the L2's +Z (dome) side, so upright it sees up and around:
+  elevation 0..90 deg in standard mode, -6..90 deg in negative-angle (wide) mode, which the PDF
+  asks for. From 0.80 m it sees the walls above the robot and the ceiling; in wide mode it
+  reaches 0.45 m-high objects only beyond about 3.1 m. It sees almost none of the robot.
   Frames (all fixed joints, published by robot_state_publisher):
-    <parent> -> l2_mount   centre of the L2's bottom mounting face, z normal to it into the
-                           sensor (dome). REWRITE: pose on the new mount.
-    l2_mount -> l2_lidar   vendor point-cloud frame. REWRITE: rotation about z that sets the
-                           cable outlet direction on the new mount.
+    <parent> -> l2_mount   centre of the L2's bottom mounting face (the standoff top), z up into
+                           the dome. 0.767 m above the floor; the housing centre (the reference
+                           URDF's unitree_l2_link) is 32.5 mm above it, at 0.799 m.
+    l2_mount -> l2_lidar   vendor point-cloud frame, rotated about z by l2_cable_yaw.
     l2_lidar -> l2_imu     vendor IMU frame: axes parallel to l2_lidar, origin at
                            (-0.007698, -0.014655, 0.00667) m in l2_lidar.
@@ -28,13 +31,24 @@
   <xacro:property name="l2_imu_y" value="-0.014655"/>
   <xacro:property name="l2_imu_z" value="0.00667"/>
+  <!-- Mount pose in base_link. x, y from the STEP body. z = STEP box top (0.7369 m above the
+       floor) + 30 mm standoff - wheel_radius.
+       STAND-IN: the height follows the PDF standoff rule, not the STEP; measure the mounted
+       L2 bottom face height. -->
+  <xacro:property name="l2_mount_x" value="-0.100"/>
+  <xacro:property name="l2_mount_y" value="0.0"/>
+  <xacro:property name="l2_mount_z" value="${0.7369 + 0.030 - wheel_radius}"/>
+  <xacro:property name="l2_standoff_height" value="0.030"/>
+  <!-- STAND-IN: cable direction unknown. 0 = vendor +X forward, cable outlet to the rear.
+       Read it on the robot (vendor +X points away from the cable) and set the yaw from
+       above, counter-clockwise positive. -->
+  <xacro:property name="l2_cable_yaw" value="0.0"/>
   <xacro:macro name="unitree_l2" params="prefix parent">
     <joint name="${prefix}l2_mount_joint" type="fixed">
       <parent link="${prefix}${parent}"/>
       <child link="${prefix}l2_mount"/>
-      <!-- REWRITE: origin removed. Set the L2's bottom mounting face pose on the new mount
-           (position, tilt, z into the dome). -->
+      <origin xyz="${l2_mount_x} ${l2_mount_y} ${l2_mount_z}" rpy="0 0 0"/>
     </joint>
-    <!-- Sensor mass only. REWRITE: add the L2 body visual/collision, unless the new mount's
-         meshes already contain it. -->
+    <!-- L2 body above the mounting face and the standoff below it. Mass: the L2 only (the
+         standoff is counted in chassis_mass). -->
     <link name="${prefix}l2_mount">
       <xacro:box_inertia mass="${l2_mass}" x="${l2_body_size}" y="${l2_body_size}"
@@ -42,4 +56,24 @@
         <origin xyz="0 0 ${l2_body_height/2}" rpy="0 0 0"/>
       </xacro:box_inertia>
+      <visual>
+        <origin xyz="0 0 ${l2_body_height/2}" rpy="0 0 0"/>
+        <geometry>
+          <box size="${l2_body_size} ${l2_body_size} ${l2_body_height}"/>
+        </geometry>
+        <material name="l2_purple"/>
+      </visual>
+      <visual>
+        <origin xyz="0 0 ${-l2_standoff_height/2}" rpy="0 0 0"/>
+        <geometry>
+          <box size="${l2_body_size} ${l2_body_size} ${l2_standoff_height}"/>
+        </geometry>
+        <material name="mount_white"/>
+      </visual>
+      <collision>
+        <origin xyz="0 0 ${(l2_body_height - l2_standoff_height)/2}" rpy="0 0 0"/>
+        <geometry>
+          <box size="${l2_body_size} ${l2_body_size} ${l2_body_height + l2_standoff_height}"/>
+        </geometry>
+      </collision>
     </link>
     <!-- Point cloud frame (vendor lidar frame) -->
@@ -47,6 +81,5 @@
       <parent link="${prefix}l2_mount"/>
       <child link="${prefix}l2_lidar"/>
-      <!-- REWRITE: rotation removed. Rotate about z so vendor +X points away from the cable
-           outlet as mounted on the new robot. -->
+      <origin xyz="0 0 0" rpy="0 0 ${l2_cable_yaw}"/>
     </joint>
     <link name="${prefix}l2_lidar"/>
@@ -59,5 +92,4 @@
     <link name="${prefix}l2_imu"/>
   </xacro:macro>
-  <!-- REWRITE: parent is base_link until the new mount's links exist -->
   <xacro:unitree_l2 prefix="$(arg prefix)" parent="base_link"/>
 </robot>

File: src/mecanum_simulation/urdf/mecanum.gazebo.xacro (robot description, xacro)
@@ -10,8 +10,9 @@
      gz:expressed_in attribute. (A bare <fdir1> under <gazebo reference> loses the attribute.)
      X-roller layout: front_left and rear_right rollers along (1, -1); front_right and
-     rear_left along (1, 1).
-     REWRITE: the fdir values below assume the previous wheels' roller handedness. Check them
-     against the new wheel meshes. The new wheel links need exactly one unnamed collision each,
-     or this friction block no longer merges and the wheels lose their mecanum behaviour.
+     rear_left along (1, 1). This matches mecanum_base/kinematics.py.
+     STAND-IN: the CAD has no rollers, so the X layout is assumed; check the roller handedness
+     on the real wheels. Each wheel link must keep exactly one unnamed collision
+     (mecanum_wheel.xacro), or this friction block no longer merges and the wheels silently
+     lose their mecanum behaviour.
   2. One JointController (velocity mode) per wheel. Its gz topic is the default
      /model/mecanum/joint/<joint>/cmd_vel (gz.msgs.Double, rad/s), bridged from
@@ -21,6 +22,7 @@
      not in the TF tree, its gz TF topic is never bridged, and nothing uses it for control or
      odometry.
-  Wheel joint states are deliberately not published: the real motors have no encoders, and
-  joint_state_publisher reports zero wheel angles in sim and on hardware alike.
+  Wheel joint states are not published: the open-loop drive reads no wheel state, and
+  joint_state_publisher reports zero wheel angles. The new motors have encoders; Phase 1 of
+  docs/plan.md moves the drive to gz_ros2_control and joint_state_broadcaster.
 -->
 <robot xmlns:xacro="http://www.ros.org/wiki/xacro" xmlns:gz="http://gazebosim.org/schema">
@@ -62,8 +64,8 @@
        The L2's field of view, in its own frame, is the hemisphere on its +Z (dome) side:
        elevation 0..90 deg in standard mode (factory default, work-mode bit 0 = 0) or
-       -6..90 deg in wide mode (bit 0 = 1). -->
-  <!-- The sensor model below is the L2's own and carries over to the new model; its pose
-       follows l2_lidar / l2_imu from the URDF. -->
-  <xacro:arg name="sim_l2_wide_fov" default="false"/>
+       -6..90 deg in wide mode (bit 0 = 1). The robot's upright mount uses wide mode (sensor
+       placement PDF: "negative-angle mode"), so it is the default here. The pose follows
+       l2_lidar / l2_imu from the URDF. -->
+  <xacro:arg name="sim_l2_wide_fov" default="true"/>
   <xacro:if value="$(arg use_l2)">
   <xacro:property name="sim_l2_min_elevation"
@@ -142,6 +144,6 @@
   </gazebo>
   </xacro:if>
-  <!-- REWRITE: add Gazebo sensors for the new model's additional sensors here, on their URDF
-       frames, and bridge them in config/gz_bridge.yaml (see REWRITE.md). -->
+  <!-- The robot's other sensors (D435i, 2D lidar, ultrasonics, cliff ToF, bumpers) are added
+       here in docs/plan.md Phase 2, on their URDF frames, and bridged in config/gz_bridge.yaml. -->
   <gazebo>
     <plugin filename="gz-sim-odometry-publisher-system"
