Commit message: Add simulated L2, self-filter and cloud-to-scan (phase 3)
- mecanum_simulation: gpu_lidar on l2_lidar (360 x 32 per sweep at
  5.55 Hz, elevation 0..90 deg in the L2 frame, wide-FOV option) and an
  IMU on l2_imu (250 Hz), bridged to /l2/points and /l2/imu: the same
  topics and frames as the real driver. World gains the Sensors and Imu
  systems and a 2.4 m ceiling.
- New mecanum_localization: pcl_ros CropBox self-filter (robot box in
  base_footprint, /l2/points -> /l2/points_filtered) and
  pointcloud_to_laserscan (0.10-0.50 m band -> /scan).
- mecanum_bringup: robot.launch.py starts perception; sensors.rviz shows
  raw and filtered clouds and the scan.

Verified in sim: all streams at 5.56 Hz, IMU 250 Hz, 25% self-hits
removed, scan matches the world; the rear is largely blind, as the
inverted 30-deg mount predicts. Stand-ins recorded in STANDINS.md.

Co-Authored-By: Claude Opus 5.5 <noreply@anthropic.com>

File: src/mecanum_simulation/urdf/mecanum.gazebo.xacro (robot description, xacro)
@@ -51,4 +51,90 @@
   <xacro:sim_mecanum_wheel wheel="rear_left" fdir="1 1 0"/>
   <xacro:sim_mecanum_wheel wheel="rear_right" fdir="1 -1 0"/>
+  <!-- 4. Simulated Unitree L2: a gpu_lidar on l2_lidar and an IMU on l2_imu, bridged to the
+       same topics and frames as the real driver (mecanum_lidar): /l2/points in l2_lidar and
+       /l2/imu in l2_imu. Requires the Sensors (ogre2) and Imu systems in the world.
+       Differences from the real L2: Gazebo renders each sweep instantaneously, so the cloud has
+       no per-point "time" field and no motion distortion; and it is a regular 360 x 32 grid
+       instead of the L2's non-repetitive pattern.
+       The L2's field of view, in its own frame, is the hemisphere on its +Z (dome) side:
+       elevation 0..90 deg in standard mode (factory default, work-mode bit 0 = 0) or
+       -6..90 deg in wide mode (bit 0 = 1). -->
+  <xacro:arg name="sim_l2_wide_fov" default="false"/>
+  <xacro:if value="$(arg use_l2)">
+  <xacro:property name="sim_l2_min_elevation"
+    value="${radians(-6.0) if '$(arg sim_l2_wide_fov)' == 'true' else 0.0}"/>
+  <gazebo reference="$(arg prefix)l2_lidar">
+    <sensor name="l2_lidar" type="gpu_lidar">
+      <gz_frame_id>$(arg prefix)l2_lidar</gz_frame_id>
+      <topic>/sim/l2/lidar</topic>
+      <!-- 5.55 Hz circumferential scan rate and 0.05..30 m range: L2 datasheet.
+           One message = one full sweep. -->
+      <update_rate>5.55</update_rate>
+      <always_on>true</always_on>
+      <visualize>false</visualize>
+      <lidar>
+        <scan>
+          <!-- STAND-IN: the L2's scan pattern is non-repetitive; 360 x 32 samples per sweep at
+               5.55 Hz gives ~64k points/s, the datasheet's effective point rate. Compare with a
+               real L2 cloud (mecanum_lidar bench test) and adjust. -->
+          <horizontal>
+            <samples>360</samples>
+            <resolution>1</resolution>
+            <min_angle>${-pi}</min_angle>
+            <max_angle>${pi}</max_angle>
+          </horizontal>
+          <vertical>
+            <samples>32</samples>
+            <resolution>1</resolution>
+            <min_angle>${sim_l2_min_elevation}</min_angle>
+            <max_angle>${pi / 2}</max_angle>
+          </vertical>
+        </scan>
+        <range>
+          <min>0.05</min>
+          <max>30.0</max>
+          <resolution>0.0045</resolution>
+        </range>
+        <noise>
+          <!-- STAND-IN: the datasheet gives accuracy <= 2.0 cm, not a noise model; 0.01 m
+               Gaussian is assumed. Measure the spread on a flat wall with the real L2. -->
+          <type>gaussian</type>
+          <mean>0.0</mean>
+          <stddev>0.01</stddev>
+        </noise>
+      </lidar>
+    </sensor>
+  </gazebo>
+  <xacro:macro name="sim_imu_noise" params="stddev">
+    <noise type="gaussian">
+      <mean>0.0</mean>
+      <stddev>${stddev}</stddev>
+    </noise>
+  </xacro:macro>
+  <gazebo reference="$(arg prefix)l2_imu">
+    <sensor name="l2_imu" type="imu">
+      <gz_frame_id>$(arg prefix)l2_imu</gz_frame_id>
+      <topic>/sim/l2/imu</topic>
+      <!-- STAND-IN: the L2 IMU output rate is not in the official datasheet (250 Hz is the
+           most quoted value); read the rate from the mecanum_lidar status line on hardware -->
+      <update_rate>250</update_rate>
+      <always_on>true</always_on>
+      <!-- STAND-IN: L2 IMU noise is unknown; typical consumer MEMS values assumed. Record the
+           IMU at rest with the real L2 and use its standard deviations. -->
+      <imu>
+        <angular_velocity>
+          <x><xacro:sim_imu_noise stddev="0.002"/></x>
+          <y><xacro:sim_imu_noise stddev="0.002"/></y>
+          <z><xacro:sim_imu_noise stddev="0.002"/></z>
+        </angular_velocity>
+        <linear_acceleration>
+          <x><xacro:sim_imu_noise stddev="0.02"/></x>
+          <y><xacro:sim_imu_noise stddev="0.02"/></y>
+          <z><xacro:sim_imu_noise stddev="0.02"/></z>
+        </linear_acceleration>
+      </imu>
+    </sensor>
+  </gazebo>
+  </xacro:if>
   <gazebo>
     <plugin filename="gz-sim-odometry-publisher-system"

Commit message: Drive the simulation through ros2_control (phase 1)
The new motors have encoders, so the sim now commands the wheels and
reads their measured state through ros2_control (decision 0002,
superseding 0001):

- New package mecanum_controllers: ros2_control xacro (hardware mock or
  sim), mecanum_drive_controller and joint_state_broadcaster config
  (wheel radius 0.1025, lx+ly 0.451, limits 0.3/0.3/0.8, 0.25 s
  reference timeout), controllers.launch.py, and a launch test on mock
  hardware that checks wheel speeds against mecanum_base/kinematics.py,
  the odometry, the limits and the timeout.
- Contract: every velocity source publishes TwistStamped on /cmd_vel;
  the controller publishes /wheel/odometry and owns odom ->
  base_footprint until the EKF (phase 3). LIO moves to /lio/odom
  without TF in sim; the hardware path keeps the open-loop driver.
- Simulation: gz_ros2_control replaces the JointController blocks;
  sim.launch.py spawns the controllers after the robot. Delete
  sim_motor_plant, plant_model, sim_plant.yaml, the wheel command
  bridges, the driver's sim transport and MotorCommands.msg.
- motion_test publishes stamped by default.
- docs: phase 1 results in plan.md (forward/strafe 99%, rotation 100%
  with 5.7 cm translation from the stand-in COM offset, wheel odometry
  loop max 0.39%, LIO 0.23%), encoder guide status, STANDINS rows and
  READMEs.

Co-Authored-By: Claude Opus 5.5 <noreply@anthropic.com>

File: src/mecanum_simulation/urdf/mecanum.gazebo.xacro (robot description, xacro)
@@ -15,14 +15,13 @@
      (mecanum_wheel.xacro), or this friction block no longer merges and the wheels silently
      lose their mecanum behaviour.
-  2. One JointController (velocity mode) per wheel. Its gz topic is the default
-     /model/mecanum/joint/<joint>/cmd_vel (gz.msgs.Double, rad/s), bridged from
-     /sim/wheel_cmd/<wheel> and driven by mecanum_simulation/sim_motor_plant.
+  2. The drive: ros2_control, not in this file. mecanum_sim.urdf.xacro includes
+     mecanum_controllers/urdf/mecanum.ros2_control.xacro with hardware=sim, which adds the
+     gz_ros2_control plugin. It commands the wheel joint velocities and reads their measured
+     positions and velocities from physics (ideal encoders) for joint_state_broadcaster and
+     mecanum_drive_controller.
   3. Ground truth: OdometryPublisher on gz topic /sim/ground_truth/odom, bridged to the ROS
      topic of the same name. Evaluation only: its frame labels (sim_gt_world, sim_gt_base) are
      not in the TF tree, its gz TF topic is never bridged, and nothing uses it for control or
      odometry.
-  Wheel joint states are not published: the open-loop drive reads no wheel state, and
-  joint_state_publisher reports zero wheel angles. The new motors have encoders; Phase 1 of
-  docs/plan.md moves the drive to gz_ros2_control and joint_state_broadcaster.
 -->
 <robot xmlns:xacro="http://www.ros.org/wiki/xacro" xmlns:gz="http://gazebosim.org/schema">
@@ -43,11 +42,4 @@
         </surface>
       </collision>
-    </gazebo>
-    <gazebo>
-      <plugin filename="gz-sim-joint-controller-system"
-              name="gz::sim::systems::JointController">
-        <joint_name>$(arg prefix)${wheel}_wheel_joint</joint_name>
-        <initial_velocity>0.0</initial_velocity>
-      </plugin>
     </gazebo>
   </xacro:macro>

File: src/mecanum_simulation/urdf/mecanum_sim.urdf.xacro (robot description, xacro)
@@ -1,5 +1,6 @@
 <?xml version="1.0"?>
 <!--
-  Simulation entry point: the unmodified robot description plus Gazebo-only additions.
+  Simulation entry point: the unmodified robot description plus Gazebo-only additions and
+  ros2_control on Gazebo hardware (mecanum_controllers).
   All xacro args of mecanum_description pass through (prefix, use_l2).
   The sim plugins assume prefix:="" and the model name "mecanum" (see mecanum.gazebo.xacro).
@@ -9,3 +10,5 @@
   <xacro:include filename="$(find mecanum_description)/urdf/mecanum.urdf.xacro"/>
   <xacro:include filename="$(find mecanum_simulation)/urdf/mecanum.gazebo.xacro"/>
+  <xacro:include filename="$(find mecanum_controllers)/urdf/mecanum.ros2_control.xacro"/>
+  <xacro:mecanum_ros2_control prefix="$(arg prefix)" hardware="sim"/>
 </robot>
